File: Amplifier.kicad_sch (KiCad schematic)
At the start: 80 parts, among them U1 OPA820, U5 TPA3116D2DAD, U6 OPA820, U7 OPA820, U8 GS8551

Commit message: layout finish,send manufature
Parts:
- added TP10, TP2, TP3, TP4, TP5, TP6, TP7, TP8, TP9: TestPoint_Probe, RM25:Testpoint_1.2_0.8, symbol Connector:TestPoint_Probe
- C37, C38: footprint Capacitor_SMD:C_0603_1608Metric -> Capacitor_SMD:C_1206_3216Metric
Connections:
- net ADC1_IN14: now also TP5.1
- net Amp_OUTP: now also TP6.1
- net MCU_Transmit: now also TP7.1
- net OUTNL: now also TP8.1
- net PreAmp_OUT: now also TP4.1
- net Transducer_Rx: now also TP2.1
- net Transducer_Tx: now also TP10.1
- net at C37.2, L4.1, L5.1: now also TP9.1
- net at R22.1, R23.1, R25.1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: now also TP3.1
