File: MCU.kicad_sch (KiCad schematic)
At the start: 91 parts, among them J20 Conn_01x04, J3 SWD, J4 Conn_01x04, Q1 AO3400A, SW2 NRST, SW3 BOOT0, SW4 SW, SW5 SW, SW6 SW, SW7 SW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

Commit message: layout finish,send manufature
Parts:
- D4: value LED_Blue -> LED_Yellow
- D5: value LED_Pink -> LED_White
- D6: value LED_White -> LED_Blue
- D7: value LED_Yellow -> LED_Pink
- JP1: footprint 0_RM2024:JUMPER_3_NODE -> Connector_PinHeader_1.00mm:PinHeader_1x03_P1.00mm_Vertical
Changed lines of the file:
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@@
 			)
 		)
-		(property "Value" "LED_Pink"
+		(property "Value" "LED_White"
 			(at 57.912 141.224 0)
 			(effects
@@
 			)
 		)
-		(property "Footprint" "0_RM2024:JUMPER_3_NODE"
+		(property "Footprint" "Connector_PinHeader_1.00mm:PinHeader_1x03_P1.00mm_Vertical"
 			(at 161.29 20.32 0)
 			(effects
@@
 			)
 		)
-		(property "Value" "LED_White"
+		(property "Value" "LED_Blue"
 			(at 57.404 145.034 0)
 			(effects
@@
 			)
 		)
-		(property "Value" "LED_Yellow"
+		(property "Value" "LED_Pink"
 			(at 57.658 150.622 0)
 			(effects
@@
 			)
 		)
-		(property "Value" "LED_Blue"
+		(property "Value" "LED_Yellow"
 			(at 57.15 138.684 0)
 			(effects
