File: Power.kicad_sch (KiCad schematic)
At the start: 30 parts, among them J2 PWRIn, U10 ISO_DC, U2 RY8411, U4 RS3236

Commit message: layout finish,send manufature
Parts:
- removed C24: 100u, Capacitor_SMD:C_2220_5750Metric, symbol Device:C_Small
- added C85: 47u, Capacitor_Tantalum_SMD:CP_EIA-3216-18_Kemet-A_Pad1.58x1.35mm_HandSolder, symbol Device:C_Polarized_Small
Connections:
- net 5V is gone; now on net +5V: C20.1, R2.1
- net GND: now also C85.2
- net at C21.1, C22.1, D2.1 (A1)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: now also C85.1
Other:
- moved on the sheet: D2, D3
