File: underwaterCom.kicad_pcb (KiCad board)
At the start: 2 copper layers, 203 parts, among them J2 PWRIn, J20 Conn_01x04, J3 SWD, J4 Conn_01x04, Q1 AO3400A, SW1 SW_SPDT, SW2 NRST, SW3 BOOT0, SW4 SW, SW5 SW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

Commit message: layout finish,send manufature
Parts:
- removed C24: 100u, Capacitor_SMD:C_2220_5750Metric
- added C85: 47u, Capacitor_Tantalum_SMD:CP_EIA-3216-18_Kemet-A_Pad1.58x1.35mm_HandSolder, F.Cu at (72.5, 46.7)
- added TP10: TestPoint_Probe, RM25:Testpoint_1.2_0.8, F.Cu at (19.8, 28.6)
- added TP2: TestPoint_Probe, RM25:Testpoint_1.2_0.8, F.Cu at (20.0, 35.1)
- added TP3: TestPoint_Probe, RM25:Testpoint_1.2_0.8, F.Cu at (34.0, 39.2)
- added TP4: TestPoint_Probe, RM25:Testpoint_1.2_0.8, F.Cu at (42.2, 38.3)
- added TP5: TestPoint_Probe, RM25:Testpoint_1.2_0.8, F.Cu at (38.6, 51.9)
- added TP6: TestPoint_Probe, RM25:Testpoint_1.2_0.8, F.Cu at (31.9, 34.1)
- added TP7: TestPoint_Probe, RM25:Testpoint_1.2_0.8, F.Cu at (50.4, 54.2)
- added TP8: TestPoint_Probe, RM25:Testpoint_1.2_0.8, F.Cu at (45.9, 24.5)
- added TP9: TestPoint_Probe, RM25:Testpoint_1.2_0.8, F.Cu at (30.2, 32.4)
- C37, C38: footprint Capacitor_SMD:C_0603_1608Metric -> Capacitor_SMD:C_1206_3216Metric
- D4: value LED_Blue -> LED_Yellow
- D5: value LED_Pink -> LED_White
- D6: value LED_White -> LED_Blue
- D7: value LED_Yellow -> LED_Pink
- JP1: footprint 0_RM2024:JUMPER_3_NODE -> Connector_PinHeader_1.00mm:PinHeader_1x03_P1.00mm_Vertical
- moved L1 180.8 mm to (72.6, 42.8), turned to -90 degrees
- moved D3 177.7 mm to (73.9, 50.0), turned to 90 degrees
- moved F1 175.9 mm to (84.6, 27.8), turned to 180 degrees
- moved C5 173.6 mm to (76.1, 30.4), turned to -90 degrees
- moved D1 171.7 mm to (81.4, 32.5), turned to -90 degrees
- moved U4 167.0 mm to (67.3, 52.3), turned to 180 degrees
- moved C26 162.6 mm to (63.0, 52.5), turned to 90 degrees
- moved J2 160.9 mm to (86.3, 37.1), turned to 90 degrees
- moved C23 160.7 mm to (65.4, 49.8), turned to 180 degrees
- moved D2 160.6 mm to (77.4, 50.3)
- moved C25 160.4 mm to (64.5, 52.5), turned to 90 degrees
- moved U2 159.3 mm to (78.2, 42.4), turned to 90 degrees
- moved C22 155.4 mm to (77.3, 48.0)
- moved C21 155.0 mm to (77.3, 45.6)
- moved R3 154.8 mm to (80.7, 42.9), turned to 90 degrees
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Connections:
- C20 pad 1: /Power/5V -> +5V
- R2 pad 1: /Power/5V -> +5V
Routing:
- net +5V: track 0.00 -> 251.9 mm, vias 0 -> 29
- net +3.3V: track 0.00 -> 237.0 mm, vias 0 -> 107
- net VCC: track 0.00 -> 97.1 mm
- net -5V: track 0.00 -> 94.7 mm, vias 0 -> 18
- net /MCU/PB3: track 0.00 -> 57.6 mm, vias 0 -> 2
- net /MCU/PA0: track 0.00 -> 53.1 mm
- net /MCU/PA2: track 0.00 -> 53.0 mm
- net /MCU/PC12: track 0.00 -> 50.3 mm, vias 0 -> 2
- net /MCU/PB4: track 0.00 -> 40.1 mm, vias 0 -> 2
- net /MCU/PC3: track 0.00 -> 36.6 mm
- net /MCU/PD2: track 0.00 -> 36.1 mm, vias 0 -> 2
- net Net-(U3-PB14): track 0.00 -> 33.7 mm, vias 0 -> 2
- net Net-(U3-PB13): track 0.00 -> 33.6 mm, vias 0 -> 2
- net /MCU/PA1: track 0.00 -> 32.9 mm
- net MCU_Transmit: track 0.00 -> 30.8 mm, vias 0 -> 1
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- added copper zone on F.Cu, net +3.3V
- added copper zone on In2.Cu, net +3.3V
- added copper zone on F.Cu, net +5V
- added copper zone on B.Cu, net GND
- added copper zone on F.Cu, net GND
- added copper zone on In1.Cu, net GND
- added copper zone on In2.Cu, net GND
- added copper zone on F.Cu, net Net-(BZ2-+)
- added copper zone on F.Cu, net Net-(D2-A1)
- added copper zone on F.Cu, net Net-(U2-LX)
Other:
- board outline added: 80 x 80 mm
- copper layers 2 -> 4
- board text added: "1 Pink"
- board text added: "12v IN"
- board text added: "2 Blue"
- board text added: "3 Yellow"
- board text added: "4 White"
- board text added: "5v DN DP GND"
- board text added: "BOOT0"
- board text added: "DIO CLK - +"
- board text added: "GND"
- board text added: "GND 3V3 SCL SDA"
- board text added: "I2C1"
- board text added: "NRST"
- board text added: "SWD"
- board text added: "Trans"
- board text added: "Tx Rx"
